File: pcb/dogboard.kicad_pcb (KiCad board)
At the start: 2 copper layers, 45.1 x 32.6 mm, 30 parts, among them J1 Barrel_Jack_Switch_Pin3Ring, J2 qtpy1, J3 Conn_01x02_Male, Q1 MMBT3904, Q2 MMBT3904, SW1 SW_Push, U1 LD1117S50TR_SOT223, U2 LM555xN

Commit message: pcb refactor
Parts:
- removed C3: 1uF, Capacitor_SMD:C_1206_3216Metric_Pad1.33x1.80mm_HandSolder
- removed D2: D_Schottky, Diode_SMD:D_1206_3216Metric_Pad1.42x1.75mm_HandSolder
- removed D3, D4, D5: LED, LED_SMD:LED_1206_3216Metric_Pad1.42x1.75mm_HandSolder
- removed J2: qtpy1, Module:qtpy1_reverse
- removed J3: Conn_01x02_Male, Connector_JST:JST_PH_S2B-PH-K_1x02_P2.00mm_Horizontal
- removed Q1, Q2: MMBT3904, Package_TO_SOT_SMD:SOT-23
- removed R5: 82, Resistor_SMD:R_0805_2012Metric_Pad1.20x1.40mm_HandSolder
- removed REF**: dog_better, proj_footprints:dog_better
- removed SW1: SW_Push, Button_Switch_THT:SW_PUSH-12mm
- removed TP3, TP4, TP5, TP6, TP7: TestPoint, TestPoint:TestPoint_Pad_D1.5mm
- removed U2: LM555xN, Package_DIP:DIP-8_W7.62mm
- added C10: 0.1u, _custom:CAP_0402_HandSolder, F.Cu at (151.8, 111.0)
- added C11: 0.1u, _custom:CAP_0402_HandSolder, F.Cu at (148.2, 100.6)
- added C12: 0.1u, _custom:CAP_0402_HandSolder, F.Cu at (148.2, 112.2)
- added C13: 0.1u, _custom:CAP_0402_HandSolder, F.Cu at (157.6, 104.7)
- added C14: 0.1u, _custom:CAP_0402_HandSolder, F.Cu at (152.8, 100.6)
- added C15: 0.1u, _custom:CAP_0402_HandSolder, F.Cu at (148.2, 111.0)
- added C18: 0.1u, _custom:CAP_0402_HandSolder, F.Cu at (151.8, 112.2)
- added C5: 0.1uF, _custom:CAP_0603_HandSolder, F.Cu at (158.2, 111.4)
- added C6: 1u, _custom:CAP_0603_HandSolder, F.Cu at (145.2, 103.4)
- added C7: 0.1u, _custom:CAP_0402_HandSolder, F.Cu at (145.2, 105.6)
- added C8: 0.1u, _custom:CAP_0402_HandSolder, F.Cu at (157.6, 103.5)
- added C9: 1u, _custom:CAP_0603_HandSolder, F.Cu at (145.2, 101.8)
- added D6: NeoPxl, _custom:LED_NeoPixel_0606, F.Cu at (154.8, 111.8)
- added R8: 27, _custom:R_0402_HandSolder, F.Cu at (141.9, 105.1)
- added REG1: 3.3v Linear, _custom:reg_SMD_SOT-25, F.Cu at (131.9, 97.5)
- added SW2: BOOT, _custom:button_SMD_PTS810, F.Cu at (148.2, 93.0)
- added U3: 4MB Flash, _custom:flash_SMD_XSON-8_4x4mm, F.Cu at (143.6, 109.4)
- added Y1: 12 MHz, _custom:XO_Osc_4-SMD_3.2x2.5, F.Cu at (158.2, 107.9)
- C1: footprint Capacitor_SMD:C_1206_3216Metric_Pad1.33x1.80mm_HandSolder -> _custom:CAP_0805_HandSolder
- C2: value 4.7 -> 1uF; footprint Capacitor_SMD:C_1206_3216Metric_Pad1.33x1.80mm_HandSolder -> _custom:CAP_0805_HandSolder
- C4: value 1uF -> 0.1u; footprint Capacitor_SMD:C_1206_3216Metric_Pad1.33x1.80mm_HandSolder -> _custom:CAP_0603_HandSolder
- D1: value SB130 -> ESD Protection; footprint Diode_THT:D_DO-41_SOD81_P10.16mm_Horizontal -> _custom:tvs_USB2_SOT-723
- J1: value Barrel_Jack_Switch_Pin3Ring -> USB-C / USB2.0; footprint Connector_BarrelJack:BarrelJack_CUI_PJ-102AH_Horizontal -> _custom:USB_C_Receptacle_SMD_GCT
- R1: value 47 -> 20k; footprint Resistor_SMD:R_0805_2012Metric_Pad1.20x1.40mm_HandSolder -> _custom:R_0805_HandSolder
- R2: value 10k -> 5.1k; footprint Resistor_SMD:R_0805_2012Metric_Pad1.20x1.40mm_HandSolder -> _custom:R_0603_HandSolder
- R3: value 220 -> 5.1k; footprint Resistor_SMD:R_0805_2012Metric_Pad1.20x1.40mm_HandSolder -> _custom:R_0603_HandSolder
- R4: footprint Resistor_SMD:R_0805_2012Metric_Pad1.20x1.40mm_HandSolder -> _custom:R_0805_HandSolder
- R6: value 150 -> 1k; footprint Resistor_SMD:R_1206_3216Metric_Pad1.30x1.75mm_HandSolder -> _custom:R_0805_HandSolder
- R7: value 10k -> 27; footprint Resistor_SMD:R_0805_2012Metric_Pad1.20x1.40mm_HandSolder -> _custom:R_0402_HandSolder
- U1: value LD1117S50TR_SOT223 -> RP2040; footprint Package_TO_SOT_SMD:SOT-223-3_TabPin2 -> _custom:RP2040_QFN-56
- moved U1 64.5 mm to (151.3, 105.8), turned to 90 degrees
- moved C4 61.2 mm to (140.2, 109.4)
- moved J1 58.4 mm to (127.8, 106.9)
- moved D1 54.5 mm to (135.6, 106.4)
- moved C1 54.2 mm to (135.3, 97.5)
- moved R2 52.5 mm to (135.6, 109.3)
- moved R6 51.8 mm to (153.0, 93.0), turned to -90 degrees
- moved R4 51.7 mm to (155.8, 93.0)
- moved C2 49.0 mm to (128.5, 97.5), turned to 90 degrees
- moved R3 44.3 mm to (135.6, 103.5)
- moved R7 41.0 mm to (141.9, 104.1), turned to 0 degrees
- moved R1 22.5 mm to (125.3, 99.6), turned to 90 degrees
Connections:
- C1 pad 2: Net-(C1-Pad2) -> VBUS
- C2 pad 2: Net-(C2-Pad2) -> +3.3V
- C4 pad 2: Net-(C3-Pad2) -> +3.3V
- D1 pad 1: Net-(C3-Pad2) -> /USB_D-
- D1 pad 2: Net-(C2-Pad2) -> /USB_D+
- R1 pad 1: Net-(J2-Pad14) -> GNDPWR
- R1 pad 2: Net-(D4-Pad2) -> GNDREF
- R2 pad 1: Net-(C2-Pad2) -> /CC2
- R2 pad 2: Net-(D2-Pad2) -> GNDREF
- R3 pad 1: Net-(C2-Pad2) -> /CC1
- R3 pad 2: Net-(D3-Pad2) -> GNDREF
- R4 pad 1: Net-(J2-Pad10) -> /~{BOOT}
- R4 pad 2: Net-(J2-Pad2) -> +3.3V
- R6 pad 2: Net-(R6-Pad2) -> /~{BOOT}
- R7 pad 1: Net-(J2-Pad13) -> /USB_D-
- R7 pad 2: Net-(J2-Pad10) -> /TR-
- U1 pad 1: GNDREF -> +3.3V
- U1 pad 2: Net-(C2-Pad2) -> GPIO0
- U1 pad 3: Net-(C1-Pad2) -> GPIO1
Routing:
- net GNDREF: track 248.0 -> 3.86 mm, vias 0 -> 1
- net Net-(J2-Pad13): track 107.5 -> 0.00 mm
- net Net-(J2-Pad11): track 73.8 -> 0.00 mm
- net Net-(J2-Pad12): track 72.6 -> 0.00 mm
- net Net-(C3-Pad2): track 57.2 -> 0.00 mm
- net Net-(J2-Pad10): track 50.8 -> 0.00 mm
- net Net-(J2-Pad2): track 50.6 -> 0.00 mm, vias 1 -> 0
- net Net-(J2-Pad14): track 45.6 -> 0.00 mm, vias 1 -> 0
- net Net-(D2-Pad1): track 40.9 -> 0.00 mm, vias 1 -> 0
- net +3.3V: track 0.00 -> 40.4 mm, vias 0 -> 4
- net Net-(J2-Pad3): track 36.3 -> 0.00 mm
- net Net-(C2-Pad2): track 36.2 -> 0.00 mm
- net Net-(J2-Pad4): track 29.6 -> 0.00 mm
- net Net-(J2-Pad5): track 28.6 -> 0.00 mm
- net Net-(J2-Pad6): track 22.8 -> 0.00 mm
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- added copper zone on F.Cu, net GNDPWR
- added copper zone on B.Cu, net GNDREF
- added copper zone on F.Cu, net GNDREF
- added copper zone on In1.Cu, net GNDREF
- added copper zone on In2.Cu, net GNDREF
- added copper zone on In3.Cu, net GNDREF
- added copper zone on In4.Cu, net GNDREF
Other:
- board size 45.1 x 32.6 mm -> 50 x 30 mm
- copper layers 2 -> 6
- board text removed: "ACT"
- board text removed: "CPU"
- board text removed: "DogBoard 1.0 BETA 2"
- board text removed: "EXT"

Commit message: rework power regulator
Parts:
- added C3: 1uF, _custom:CAP_0805_HandSolder, F.Cu at (137.8, 92.6)
- added R5: 120, _custom:R_1206_HandSolder, F.Cu at (126.3, 94.0)
- C1: value 1uF -> 150uF; footprint _custom:CAP_0805_HandSolder -> _custom:CAP_Tantalum_2312
- R1: value 20k -> 10k; footprint _custom:R_0805_HandSolder -> _custom:R_1206_HandSolder
- SW2: footprint _custom:button_SMD_PTS810 -> _custom:button_metal_smd
- moved SW2 18.9 mm to (130.0, 87.9)
- moved R4 17.7 mm to (139.1, 87.2)
- moved R6 17.7 mm to (136.3, 87.2)
- moved C2 9.49 mm to (137.8, 99.4), turned to 180 degrees
- moved REG1 6.09 mm to (137.8, 96.0), turned to 90 degrees
- moved C1 5.19 mm to (130.3, 96.1), turned to 90 degrees
- moved R1 1.12 mm to (126.3, 99.1)
- turned R2 to -90 degrees
- turned R3 to 90 degrees
Connections:
- C1 pad 1: GNDREF -> VBUS
- C1 pad 2: VBUS -> Net-(C1-Pad2)
- C2 pad 2: +3.3V -> VBUS
Routing:
- net GNDREF: track 3.86 -> 6.71 mm
- net +3.3V: track 40.4 -> 43.0 mm

Commit message: PBC rev 2 beta-1
Parts:
- added C16: 1uF, _custom:CAP_0805_HandSolder, F.Cu at (135.1, 100.2)
- added C17: 1uF, _custom:CAP_0805_HandSolder, F.Cu at (141.9, 100.2)
- added C19: 1uF, _custom:CAP_0603_HandSolder, F.Cu at (143.5, 86.5)
- added C20: 1uF, _custom:CAP_0603_HandSolder, F.Cu at (169.5, 86.5)
- added D10: LED_NeoPixel, _custom:LED_NeoPixel_0606, F.Cu at (146.0, 86.5)
- added D12: MP-LED, _custom:LED_MP-Cathode_1113, F.Cu at (154.9, 91.8)
- added D13: MP-LED, _custom:LED_MP-Cathode_1113, F.Cu at (160.9, 91.8)
- added D2: LED_NeoPixel, _custom:LED_NeoPixel_0606, F.Cu at (167.0, 86.5)
- added D3: LED_NeoPixel, _custom:LED_NeoPixel_0606, F.Cu at (164.0, 86.5)
- added D4: LED_NeoPixel, _custom:LED_NeoPixel_0606, F.Cu at (161.0, 86.5)
- added D5: LED_NeoPixel, _custom:LED_NeoPixel_0606, F.Cu at (158.0, 86.5)
- added D7: LED_NeoPixel, _custom:LED_NeoPixel_0606, F.Cu at (155.0, 86.5)
- added D8: LED_NeoPixel, _custom:LED_NeoPixel_0606, F.Cu at (152.0, 86.5)
- added D9: LED_NeoPixel, _custom:LED_NeoPixel_0606, F.Cu at (149.0, 86.5)
- added J2: Lights, _custom:conn_1x02_JST_PH_P2.00mm_THT_Horizontal, F.Cu at (169.0, 98.5)
- added J3: Current Conn, Connector_PinHeader_2.54mm:PinHeader_1x02_P2.54mm_Vertical, F.Cu at (170.8, 93.0)
- added R10: 10k, _custom:R_0805_HandSolder, F.Cu at (146.7, 90.9)
- added R11: 15k, _custom:R_0805_HandSolder, F.Cu at (162.0, 96.4)
- added R12: 10k, _custom:R_0805_HandSolder, F.Cu at (146.7, 95.4)
- added SW1: BOOT, _custom:button_metal_smd, F.Cu at (130.0, 87.9)
- added SW3: Action, _custom:button_SMD_PTS810, F.Cu at (142.4, 95.4)
- added U2: L9110H, _custom:GenericIC_TH-DIP-8, F.Cu at (167.0, 108.0)
- added U4: BCR430, _custom:BCR430_CC_LED_Driver, F.Cu at (162.0, 99.8)
- C1: value 150uF -> 10uF; footprint _custom:CAP_Tantalum_2312 -> _custom:CAP_1206_NoKeepout
- C2, C3: value 1uF -> 10uF; footprint _custom:CAP_0805_HandSolder -> _custom:CAP_1206_NoKeepout
- SW2: value BOOT -> Action; footprint _custom:button_metal_smd -> _custom:button_SMD_PTS810
- moved SW2 12.8 mm to (142.4, 90.9), turned to 180 degrees
- moved C2 7.52 mm to (131.0, 96.2)
- moved C3 6.83 mm to (131.0, 93.2), turned to 180 degrees
- moved REG1 4.26 mm to (138.5, 100.2)
- moved C1 3.18 mm to (131.0, 99.2), turned to 180 degrees
- moved R4 2.37 mm to (137.0, 86.1), turned to 180 degrees
- moved R6 1.30 mm to (137.0, 88.3), turned to 0 degrees
- moved R2 0.94 mm to (136.3, 108.7), turned to 0 degrees
- moved R3 0.94 mm to (136.3, 104.1), turned to 0 degrees
- moved D1 0.71 mm to (136.3, 106.4)
- moved C5 0.25 mm to (158.4, 111.2)
- moved C6 0.25 mm to (145.3, 103.2)
- moved C9 0.25 mm to (145.3, 101.6)
- moved U1 0.25 mm to (151.5, 105.6)
- moved Y1 0.25 mm to (158.4, 107.7)
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Connections:
- C1 pad 2: Net-(C1-Pad2) -> /GND_RET
- C2 pad 1: GNDREF -> VBUS
- C2 pad 2: VBUS -> /GND_RET
- C3 pad 1: GNDREF -> VBUS
- C3 pad 2: +3.3V -> /GND_RET
- R5 pad 1: Net-(C1-Pad2) -> /GND_RET
- SW2 pad 1: Net-(R6-Pad1) -> /BTN_{ACT}
- U1 pad 17: GPIO14 -> /SIG_{A}
- U1 pad 18: GPIO15 -> /SIG_{B}
- U1 pad 38: GPIO26 -> /BTN_{ACT}
- U1 pad 39: GPIO27 -> /BTN_{SET}
Routing:
- net /~{BOOT}: track 9.29 -> 38.8 mm, vias 0 -> 2
- net GPIO17: track 0.00 -> 24.3 mm, vias 0 -> 2
- net V_{SS}: track 0.00 -> 21.2 mm
- net /OUT_{B}: track 0.00 -> 19.9 mm
- net /OUT_{A}: track 0.00 -> 18.6 mm
- net /BTN_{ACT}: track 0.00 -> 18.2 mm
- net /SIG_{B}: track 0.00 -> 17.9 mm, vias 0 -> 1
- net /SIG_{A}: track 0.00 -> 14.9 mm, vias 0 -> 1
- net /USB_D+: track 0.00 -> 13.9 mm
- net /USB_D-: track 0.00 -> 13.9 mm
- net /BTN_{SET}: track 0.00 -> 13.6 mm
- net Net-(R6-Pad1): track 0.00 -> 9.60 mm
- net /OUT_{C}: track 0.00 -> 8.69 mm
- net +3.3V: track 43.0 -> 51.5 mm, vias 4 -> 12
- net GNDREF: track 6.71 -> 13.0 mm, vias 1 -> 26
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- added copper zone on B.Cu, net +3.3V
- added copper zone on F.Cu, net +3.3V
- added copper zone on In2.Cu, net +3.3V
- added copper zone on In4.Cu, net +3.3V
- added copper zone on F.Cu, net /GND_RET
- added copper zone on F.Cu, net /OUT_{B}
- added copper zone on F.Cu, net /OUT_{C}
- added copper zone on F.Cu, net VBUS
- added copper zone on In3.Cu, net VBUS
- removed copper zone on In2.Cu, net GNDREF
- removed copper zone on In3.Cu, net GNDREF
Other:
- board text added: "2.0 BETA 1"
- board text added: "A"
- board text added: "B"

Commit message: PCB rev 2 beta-2
Parts:
- moved SW1 0.50 mm to (129.5, 87.9)
- moved R4 0.40 mm to (136.6, 86.1)
- moved R6 0.40 mm to (136.6, 88.3)
- turned D12 to 180 degrees
Connections:
- D12 pad 1: /OUT_{C} -> /OUT_{B}
- D12 pad 2: /OUT_{B} -> /OUT_{C}
Other:
- board text added: "2.0 BETA 2"
- board text removed: "2.0 BETA 1"

Commit message: dogboard-2b3
Parts:
- removed C19, C20: 1uF, _custom:CAP_0603_HandSolder
- removed D10, D2, D3, D4, D5, D7, D8, D9: LED_NeoPixel, _custom:LED_NeoPixel_0606
- removed R12: 10k, _custom:R_0805_HandSolder
- removed SW1: BOOT, _custom:button_metal_smd
- added H1: MountingHole, _custom:MountingHole_M2.5, F.Cu at (128.0, 88.0)
- added H2: MountingHole, _custom:MountingHole_M2.5, F.Cu at (170.0, 88.0)
- added H3: MountingHole, _custom:MountingHole_M2.5, F.Cu at (170.0, 116.0)
- added H4: MountingHole, _custom:MountingHole_M2.5, F.Cu at (128.0, 116.0)
- added JP1: Boot-Jumper, _custom:Jumper_Open_SMD_3.5mm, F.Cu at (135.3, 112.2)
- added Q1: MOSFET, _custom:GenericIC_SOT-363, F.Cu at (154.7, 96.8)
- added Q2: MOSFET, _custom:GenericIC_SOT-363, F.Cu at (151.2, 96.8)
- added Q3: N-MOS, _custom:Transistor_SOT-323, F.Cu at (147.8, 96.8)
- added R9: 10k, _custom:R_Array_4x1206_Convex, F.Cu at (158.6, 101.0)
- C1: value 10uF -> 150uF; footprint _custom:CAP_1206_NoKeepout -> _custom:CAP_Tantalum_2312
- C2: value 10uF -> 10u
- C3: value 10uF -> 0.1u; footprint _custom:CAP_1206_NoKeepout -> _custom:CAP_0402_HandSolder
- R10: footprint _custom:R_0805_HandSolder -> _custom:R_Array_4x1206_Convex
- R4, R6: footprint _custom:R_0805_HandSolder -> _custom:R_0603_HandSolder
- U3: value 4MB Flash -> 8MB Flash
- moved C2 31.7 mm to (162.7, 95.9), turned to 90 degrees
- moved C3 28.5 mm to (157.5, 103.7), turned to 0 degrees
- moved R4 25.7 mm to (140.3, 111.5), turned to -90 degrees
- moved R6 23.3 mm to (138.5, 111.5), turned to -90 degrees
- moved SW3 7.60 mm to (134.8, 95.3), turned to -90 degrees
- moved J3 7.36 mm to (164.5, 89.2)
- moved R10 6.53 mm to (143.9, 96.8)
- moved D12 6.04 mm to (150.2, 88.0)
- moved D13 6.04 mm to (156.2, 88.0)
- moved SW2 5.33 mm to (139.4, 95.3), turned to -90 degrees
- moved R11 4.81 mm to (158.5, 93.1), turned to 0 degrees
- moved U4 4.68 mm to (158.5, 96.7), turned to -90 degrees
- moved C1 2.53 mm to (130.2, 96.8), turned to 90 degrees
- moved J2 1.58 mm to (168.5, 97.0)
- moved C8 1.51 mm to (157.5, 104.8)
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Connections:
- net /OUT_{A} renamed /Output/OUT_{A}
- net /OUT_{B} renamed /Output/OUT_{B}
- net /OUT_{C} renamed /Output/OUT_{C}
- C2 pad 2: /GND_RET -> GNDREF
- C3 pad 1: VBUS -> +3.3V
- C3 pad 2: /GND_RET -> GNDREF
- R6 pad 1: Net-(R6-Pad1) -> /~{BOOT}
- R6 pad 2: /~{BOOT} -> Net-(JP1-A)
- U1 pad 17: /SIG_{A} -> GPIO14
- U1 pad 18: /SIG_{B} -> GPIO15
- U1 pad 38: /BTN_{ACT} -> GPIO26
- U1 pad 39: /BTN_{SET} -> SIG_{A}
- U1 pad 4: GPIO2 -> /BTN_{ACT}
- U1 pad 40: GPIO28 -> SIG_{B}
- U1 pad 7: GPIO5 -> /BTN_{SET}
- U2 pad 6: /SIG_{A} -> /Output/LVL_{A}
- U2 pad 7: /SIG_{B} -> /Output/LVL_{B}
Routing:
- net /Output/LVL_{B}: track 0.00 -> 28.8 mm, vias 0 -> 1
- net /~{BOOT}: track 39.0 -> 13.5 mm, vias 2 -> 0
- net /Output/LVL_{A}: track 0.00 -> 24.8 mm, vias 0 -> 1
- net GPIO17: track 24.3 -> 0.00 mm, vias 2 -> 0
- net /BTN_{SET}: track 13.6 -> 35.2 mm, vias 0 -> 2
- net V_{SS}: track 21.2 -> 0.00 mm
- net /SIG_{B}: track 17.9 -> 0.00 mm, vias 1 -> 0
- net /SIG_{A}: track 14.9 -> 0.00 mm, vias 1 -> 0
- net SIG_{A}: track 0.00 -> 11.5 mm, vias 0 -> 2
- net /Output/OUT_{A}: track 18.6 -> 29.7 mm
- net Net-(R6-Pad1): track 9.55 -> 0.00 mm
- net Net-(Q2A-G_{A}): track 0.00 -> 9.33 mm, vias 0 -> 2
- net /Output/OUT_{C}: track 8.69 -> 0.00 mm
- net Net-(Q2A-D_{A}): track 0.00 -> 8.08 mm
- net /Output/OUT_{B}: track 19.9 -> 27.7 mm
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- added copper zone on F.Cu, net V_{SS}
- removed copper zone on B.Cu, net +3.3V
- removed copper zone on In4.Cu, net +3.3V
Other:
- board size 50 x 30 mm -> 50 x 36 mm
- board text added: "2.0 BETA 3"
- board text added: "ACT"
- board text added: "SET"
- board text removed: "2.0 BETA 2"

Commit message: pcb updates
Parts:
- removed Q3: N-MOS, _custom:Transistor_SOT-323
- added C19: 0.1uF, _custom:CAP_0402_HandSolder, F.Cu at (146.4, 92.3)
- added C20: 1uF, _custom:CAP_0603_HandSolder, F.Cu at (146.7, 97.5)
- added U5: PCA9685, _custom:GenericIC_VQFN-28-EP-6x6mm, F.Cu at (152.0, 95.4)
- C2: value 10u -> 4.7u; footprint _custom:CAP_1206_NoKeepout -> _custom:CAP_0805_NoKeepout
- moved C2 22.6 mm to (162.0, 118.5), turned to 180 degrees
- moved R11 22.4 mm to (158.1, 115.5), turned to 90 degrees
- moved U4 19.1 mm to (162.0, 115.5), turned to 0 degrees
- moved Q2 7.24 mm to (158.4, 97.6), turned to 0 degrees
- moved R9 5.59 mm to (162.5, 97.0), turned to 0 degrees
- moved Q1 4.45 mm to (158.4, 94.4), turned to 0 degrees
- moved R10 0.82 mm to (143.7, 96.0), turned to 0 degrees
Connections:
- Q2 pad 2: Net-(Q2A-G_{A}) -> SIG_{B}
- R10 pad 1: /BTN_{ACT} -> +3.3V
- R10 pad 2: +3.3V -> SCL
- R10 pad 3: /BTN_{SET} -> +3.3V
- R10 pad 4: +3.3V -> SDA
- R10 pad 5: unconnected-(R10-Pad5) -> /BTN_{ACT}
- R10 pad 6: unconnected-(R10-Pad6) -> +3.3V
- R10 pad 7: +3.3V -> /BTN_{SET}
- R10 pad 8: Net-(Q2A-G_{A}) -> +3.3V
- R9 pad 1: Net-(Q2A-D_{A}) -> Net-(Q1A-D_{A})
- R9 pad 3: Net-(Q1A-D_{A}) -> Net-(Q2A-D_{A})
- R9 pad 5: /Output/LVL_{B} -> /Output/LVL_{A}
- R9 pad 7: /Output/LVL_{A} -> /Output/LVL_{B}
- U1 pad 15: SDA -> unconnected-(U1-GPIO12-Pad15)
- U1 pad 16: SCL -> unconnected-(U1-GPIO13-Pad16)
- U1 pad 39: SIG_{A} -> SDA
- U1 pad 40: SIG_{B} -> SCL
Routing:
- net /Output/LVL_{B}: track 28.8 -> 0.00 mm, vias 1 -> 0
- net /Output/LVL_{A}: track 24.8 -> 0.00 mm, vias 1 -> 0
- net SIG_{A}: track 11.5 -> 0.00 mm, vias 2 -> 0
- net Net-(Q2A-G_{A}): track 9.33 -> 0.00 mm, vias 2 -> 0
- net /BTN_{SET}: track 35.2 -> 26.2 mm
- net Net-(Q2A-D_{A}): track 8.08 -> 0.00 mm
- net Net-(Q1A-D_{A}): track 6.66 -> 0.00 mm
- net +3.3V: track 55.0 -> 48.4 mm
- net SIG_{B}: track 5.82 -> 0.00 mm
- net /BTN_{ACT}: track 24.0 -> 21.8 mm
- net GNDREF: track 9.51 -> 10.3 mm

Commit message: dogboard-2b4
Parts:
- removed C19: 0.1uF, _custom:CAP_0402_HandSolder
- removed D1: ESD Protection, _custom:tvs_USB2_SOT-723
- removed R9: 10k, _custom:R_Array_4x1206_Convex
- added J4: i2c, _custom:conn_1x04mp_JST_SH_Micro_P1.00mm_Horizontal, F.Cu at (135.3, 116.7)
- added R12: 10k, _custom:R_0603_HandSolder, F.Cu at (161.4, 93.1)
- added R13: 10k, _custom:R_0603_HandSolder, F.Cu at (161.4, 96.2)
- added R14: 10k, _custom:R_0603_HandSolder, F.Cu at (159.5, 99.7)
- added R15: 10k, _custom:R_0603_HandSolder, F.Cu at (157.8, 99.7)
- moved Q2 1.43 mm to (158.7, 96.2)
- moved Q1 1.33 mm to (158.7, 93.1)
- moved C14 1.00 mm to (153.0, 100.4), turned to 0 degrees
- moved C20 0.20 mm to (146.7, 97.3)
Connections:
- U1 pad 15: unconnected-(U1-GPIO12-Pad15) -> GPIO12
- U1 pad 16: unconnected-(U1-GPIO13-Pad16) -> GPIO13
- U1 pad 17: GPIO14 -> UART_{RX}
- U1 pad 18: GPIO15 -> UART_{TX}
- U1 pad 37: GPIO25 -> SCL
- U1 pad 38: GPIO26 -> SDA
- U1 pad 39: SDA -> GPIO27
- U1 pad 40: SCL -> GPIO28
- U5 pad 12: unconnected-(U5-LED8-Pad12) -> SIG_{B}
- U5 pad 14: unconnected-(U5-LED10-Pad14) -> SIG_{A}
Routing:
- net UART_{TX}: track 0.00 -> 23.6 mm, vias 0 -> 2
- net UART_{RX}: track 0.00 -> 22.5 mm, vias 0 -> 2
- net SCL: track 0.00 -> 15.7 mm, vias 0 -> 2
- net /Output/LVL_{A}: track 0.00 -> 14.6 mm, vias 0 -> 1
- net /Output/LVL_{B}: track 0.00 -> 13.9 mm, vias 0 -> 1
- net SDA: track 0.00 -> 13.7 mm, vias 0 -> 2
- net +3.3V: track 48.4 -> 57.8 mm
- net /BTN_{SET}: track 26.2 -> 34.2 mm
- net GNDREF: track 10.3 -> 17.7 mm, vias 19 -> 31
- net V_{SS}: track 0.00 -> 5.36 mm
- net VBUS: track 11.1 -> 14.8 mm, vias 10 -> 13
- net SIG_{B}: track 0.00 -> 3.55 mm
- net SIG_{A}: track 0.00 -> 3.09 mm
- net /BTN_{ACT}: track 21.8 -> 24.6 mm
- net Net-(Q2A-D_{A}): track 0.00 -> 2.51 mm
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Other:
- board text added: "2.0 BETA 4"
- board text removed: "2.0 BETA 3"

Commit message: New board revision
Parts:
- moved C11 0.10 mm to (148.3, 100.4)
- moved C14 0.10 mm to (153.1, 100.4)
Connections:
- U1 pad 15: GPIO12 -> UART_{TX}
- U1 pad 16: GPIO13 -> UART_{RX}
- U1 pad 17: UART_{RX} -> GPIO14
- U1 pad 18: UART_{TX} -> GPIO15
- U1 pad 36: GPIO24 -> SDA
- U1 pad 38: SDA -> GPIO26
Routing:
- net GNDREF: track 17.7 -> 23.5 mm
- net /BTN_{ACT}: track 24.6 -> 24.0 mm
Other:
- board text added: "2.0 BETA 5"
- board text removed: "2.0 BETA 4"
